File: AQ32_v2/AQ32_v2.sch (EAGLE design)
At the start: 113 parts, among them Q2 BCV27, Q3 BCV27, Q5 BCV27, Q6 BCV27, U1 ITG-3200, U10 MS5611, U11 MIC5239, U13 74AHC1G86DCK, U2 STM32F10XVXT6, U7 USD-SOCKETNEW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

Commit message: relocated BM input away from 3.3V input, added more clearance between mounting holes and USB input, added XOR gate to SBUS TX, added ground plane to top side of board
Parts:
- added JP1: (no value), SparkFun-Connectors:M02PTH
- added U3: 74AHC1G86DCK, 74xx-little-us:74AHC1G86DCK
Connections:
- new net PD8: U2PORTD_H.PD8, U3A.O
- net 3V3AN: now also JP1-2.7, JP1-2.8
- net 3V3DIG: now also U3P.VCC; no longer JP1-2.8
- net GND: now also JP1.1, U3P.GND
- net LIPO: now also JP1.2; no longer JP1-2.7
- net NSS2_LV: now also U3A.I1
- net UART3_TX: now also U3A.I0; no longer U2PORTD_H.PD8
Other:
- moved on the sheet: C8, I2C-1, I2C-2, I2C-3, I2C-4, R1, R3, R64, SERIAL-1, SERIAL-2, SERIAL-3, SERIAL-4
