File: AQ32_v2/AQ32_v2.sch (EAGLE design)
At the start: 116 parts, among them Q2 BCV27, Q3 BCV27, Q5 BCV27, Q6 BCV27, U1 ITG-3200, U10 MS5611, U11 MIC5239, U13 74AHC1G86DCK, U2 STM32F10XVXT6, U3 74AHC1G86DCK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

Commit message: Latest from Alfred (20130526_b)
Parts:
- added C2: 0.1uF, SparkFun:CAP0402
- C42: value 220uF -> 47uF
- C44: value 47uF -> 220uF
Connections:
- net 3V3DIG: now also C2.1
- net GND: now also C2.2
Changed lines of the file:
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@@
 <part name="R8" library="rcl" deviceset="R-US_" device="R0402" value="10k"/>
 <part name="R60" library="rcl" deviceset="R-US_" device="R0402" value="10k"/>
-<part name="C42" library="rcl" deviceset="C-US" device="C0805" value="220uF"/>
+<part name="C42" library="rcl" deviceset="C-US" device="C0805" value="47uF"/>
 <part name="C43" library="rcl" deviceset="C-US" device="C0805" value="10uF"/>
-<part name="C44" library="rcl" deviceset="C-US" device="C1206" value="47uF"/>
+<part name="C44" library="rcl" deviceset="C-US" device="C1206" value="220uF"/>
 <part name="U10" library="DSP-TI" deviceset="MS5611" device=""/>
 <part name="SUPPLY19" library="supply2" deviceset="GND" device=""/>
@@
 <part name="P+4" library="SparkFun" deviceset="3.3V" device="" value="VDDA"/>
 <part name="R39" library="SparkFun" deviceset="RESISTOR" device="0402" value="0R"/>
+<part name="C2" library="SparkFun" deviceset="CAP" device="0402" value="0.1uF"/>
 </parts>
 <sheets>
@@
 <instance part="P+4" gate="G$1" x="309.88" y="58.42"/>
 <instance part="R39" gate="G$1" x="22.86" y="81.28" rot="R90"/>
+<instance part="C2" gate="G$1" x="88.9" y="170.18"/>
 </instances>
 <busses>
@@
 <pinref part="C39" gate="G$1" pin="2"/>
 <pinref part="C40" gate="G$1" pin="2"/>
+<wire x1="81.28" y1="167.64" x2="88.9" y2="167.64" width="0.1524" layer="91"/>
+<pinref part="C2" gate="G$1" pin="2"/>
 </segment>
 <segment>
@@
 <pinref part="C40" gate="G$1" pin="1"/>
 <label x="83.82" y="175.26" size="1.778" layer="95"/>
-</segment>
-<segment>
+<pinref part="C2" gate="G$1" pin="1"/>
+<wire x1="81.28" y1="175.26" x2="88.9" y2="175.26" width="0.1524" layer="91"/>
+</segment>
+<segment>
