File: AQ32_v2/AQ32_v2.brd (EAGLE design)
At the start: 57.1 x 57.1 mm, 117 parts, among them Q2 BCV27, Q3 BCV27, Q5 BCV27, Q6 BCV27, U1 ITG-3200, U10 MS5611, U11 MIC5239, U13 74AHC1G86DCK, U2 STM32F10XVXT6, U3 74AHC1G86DCK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

Commit message: change LED connector type for normal 100mil pitch
Parts:
- JP1, JP4-1, JP4-2: device SparkFun-Connectors:1X02_LOCK -> SparkFun-Connectors:1X02
- moved JP1 0.19 mm to (5.08, 45.7)
- moved JP4-1 0.18 mm to (2.54, 43.2)
- moved JP4-2 0.18 mm to (2.54, 40.6)
Changed lines of the file:
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@@
 <setting verticaltext="up"/>
 </settings>
-<grid distance="0.0125" unitdist="inch" unit="inch" style="lines" multiple="2" display="yes" altdistance="0.01" altunitdist="mm" altunit="mm"/>
+<grid distance="0.01" unitdist="inch" unit="inch" style="lines" multiple="2" display="yes" altdistance="0.01" altunitdist="mm" altunit="mm"/>
 <layers>
 <layer number="1" name="Top" color="4" fill="1" visible="yes" active="yes"/>
@@
 <element name="OSD" library="con-jst2" package="SM07B-SRSS-TB" value="SM07B-SRSS-TB" x="54.61" y="41.91" rot="R90"/>
 <element name="L2" library="SparkFun" package="0805" value="22uH" x="34.544" y="45.72" rot="R90"/>
-<element name="JP4-1" library="SparkFun-Connectors" package="1X02_LOCK" value="JP4" x="2.667" y="43.307"/>
-<element name="JP4-2" library="SparkFun-Connectors" package="1X02_LOCK" value="JP4" x="2.667" y="40.767"/>
+<element name="JP4-1" library="SparkFun-Connectors" package="1X02" value="JP4" x="2.537" y="43.177"/>
+<element name="JP4-2" library="SparkFun-Connectors" package="1X02" value="JP4" x="2.537" y="40.6375"/>
 <element name="JP3-1" library="SparkFun-Connectors" package="1X09" value="M09" x="2.54" y="37.465" rot="R270"/>
 <element name="JP3-2" library="SparkFun-Connectors" package="1X09" value="M09" x="5.08" y="37.465" rot="R270"/>
 <element name="JP5" library="SparkFun-Connectors" package="1X02" value="" x="45.72" y="11.43"/>
 <element name="U3" library="74xx-little-us" package="SC70-5" value="74AHC1G86DCK" x="10.16" y="31.75" rot="R180"/>
-<element name="JP1" library="SparkFun-Connectors" package="1X02_LOCK" value="JP1" x="5.21" y="45.855" rot="R180"/>
+<element name="JP1" library="SparkFun-Connectors" package="1X02" value="JP1" x="5.08" y="45.715" rot="R180"/>
 </elements>
 <signals>
@@
 <wire x1="6.6354" y1="38.1321" x2="5.6515" y2="39.116" width="0.4064" layer="1"/>
 <wire x1="5.6515" y1="39.116" x2="4.0132" y2="39.116" width="0.4064" layer="1"/>
-<wire x1="4.0132" y1="39.116" x2="2.4892" y2="40.767" width="0.4064" layer="1"/>
+<wire x1="4.0132" y1="39.116" x2="2.537" y2="40.6375" width="0.4064" layer="1"/>
 </signal>
 <signal name="LEDGND1">
@@
 <contactref element="Q2" pad="3"/>
 <wire x1="9.8855" y1="41.5925" x2="7.493" y2="41.5925" width="0.4064" layer="1"/>
-<wire x1="7.493" y1="41.5925" x2="6.4135" y2="42.037" width="0.4064" layer="1"/>
-<wire x1="6.4135" y1="42.037" x2="3.6322" y2="42.037" width="0.3048" layer="1"/>
-<wire x1="3.6322" y1="42.037" x2="2.4892" y2="43.307" width="0.4064" layer="1"/>
+<wire x1="7.493" y1="41.5925" x2="6.5435" y2="41.907" width="0.4064" layer="1"/>
+<wire x1="6.5435" y1="41.907" x2="3.7622" y2="41.907" width="0.3048" layer="1"/>
+<wire x1="3.7622" y1="41.907" x2="2.537" y2="43.177" width="0.4064" layer="1"/>
 </signal>
 <signal name="LEDGND2">
@@
 <wire x1="7.8535" y1="44.831" x2="7.79" y2="44.8515" width="0.4064" layer="1"/>
 <wire x1="7.79" y1="44.8515" x2="6.7945" y2="44.196" width="0.4064" layer="1"/>
-<wire x1="6.7945" y1="44.196" x2="5.3848" y2="43.307" width="0.4064" layer="1"/>
+<wire x1="6.7945" y1="44.196" x2="5.077" y2="43.177" width="0.4064" layer="1"/>
 </signal>
 <signal name="LEDGND4">
 <contactref element="Q6" pad="3"/>
 <contactref element="JP4-2" pad="2"/>
-<wire x1="5.3848" y1="40.767" x2="7.4168" y2="39.7623" width="0.4064" layer="1"/>
+<wire x1="5.077" y1="40.6375" x2="7.4168" y2="39.7623" width="0.4064" layer="1"/>
 <wire x1="7.4168" y1="39.7623" x2="7.79" y2="38.7541" width="0.4064" layer="1"/>
 <wire x1="7.79" y1="38.5445" x2="7.79" y2="38.7541" width="0.2032" layer="1"/>
@@
 <wire x1="6.5255" y1="47.9425" x2="8.8265" y2="46.9115" width="0.2032" layer="1"/>
 <contactref element="JP1" pad="2"/>
-<wire x1="2.794" y1="47.1805" x2="2.4922" y2="45.855" width="0.254" layer="1"/>
+<wire x1="2.794" y1="47.1805" x2="2.54" y2="45.715" width="0.254" layer="1"/>
 </signal>
 <signal name="5V-2">
